File: Tandy1000-PS2-adapter.sch (KiCad schematic (older format))
At the start: 11 parts, among them J1 Mini-DIN-6, J2 Conn_01x05, U1 ATtiny85

Commit message: 1.2 Update
Enlarged mounting holes to 2.7mm for more zip-tie compatibility.
Parts:
- H1, H2: footprint MountingHole:MountingHole_2.2mm_M2_DIN965_Pad -> MountingHole:MountingHole_2.7mm_M2.5_DIN965_Pad
- U1: symbol MCU_Microchip_ATtiny:ATtiny85-20SU -> Tandy1000-PS2-adapter-rescue:ATtiny85-20SU-MCU_Microchip_ATtiny
Changed lines of the file:
@@
 $EndComp
 $Comp
-L MCU_Microchip_ATtiny:ATtiny85-20SU U1
+L Tandy1000-PS2-adapter-rescue:ATtiny85-20SU-MCU_Microchip_ATtiny U1
 U 1 1 5ECCA5F4
 P 5050 3550
@@
 F 0 "H1" V 6104 5100 50  0000 L CNN
 F 1 "MountingHole_Pad" V 6195 5100 50  0000 L CNN
-F 2 "MountingHole:MountingHole_2.2mm_M2_DIN965_Pad" H 6150 4950 50  0001 C CNN
+F 2 "MountingHole:MountingHole_2.7mm_M2.5_DIN965_Pad" H 6150 4950 50  0001 C CNN
 F 3 "~" H 6150 4950 50  0001 C CNN
 	1    6150 4950
@@
 F 0 "H2" V 6104 5350 50  0000 L CNN
 F 1 "MountingHole_Pad" V 6195 5350 50  0000 L CNN
-F 2 "MountingHole:MountingHole_2.2mm_M2_DIN965_Pad" H 6150 5200 50  0001 C CNN
+F 2 "MountingHole:MountingHole_2.7mm_M2.5_DIN965_Pad" H 6150 5200 50  0001 C CNN
 F 3 "~" H 6150 5200 50  0001 C CNN
 	1    6150 5200
